File: revised_minh_design/revised_minh_design.kicad_sch (KiCad schematic)
At the start: 17 parts

Commit message: libraries and footprints
Parts:
- C1, C2, C3: renamed from C?; footprint (none) -> Capacitor_THT:C_Disc_D6.0mm_W2.5mm_P5.00mm
- D1: renamed from D?; value D_Zener -> TZX3V6A-TR; footprint (none) -> Diode_THT:D_DO-35_SOD27_P7.62mm_Horizontal
- D2: renamed from D?; footprint (none) -> LED_THT:LED_D3.0mm_Clear
- J1: renamed from J?; footprint (none) -> Connector_PinSocket_2.54mm:PinSocket_1x03_P2.54mm_Vertical
- J2: renamed from J?; footprint (none) -> Connector_PinSocket_2.54mm:PinSocket_1x07_P2.54mm_Vertical
- R1, R2, R3, R4: renamed from R?; footprint (none) -> Resistor_THT:R_Axial_DIN0309_L9.0mm_D3.2mm_P15.24mm_Horizontal
- U1: renamed from U?; footprint (none) -> Library:ESP32-devkitC-v4
- U3: renamed from U?; footprint (none) -> Package_DIP:DIP-8_W7.62mm
- U4: renamed from U?; footprint (none) -> Library:CB101
- gave numbers to parts that had none: 1
