File: board1_Arduino_ADC_DAC/revised_minh_design.kicad_pcb (KiCad board)
At the start: 4 copper layers, 96 x 43.9 mm, 40 parts, among them J1 Conn_01x03_Male, J2 Conn_02x08_Odd_Even, J3 Conn_02x08_Odd_Even, J4 Conn_02x08_Odd_Even, J5 Conn_01x02_Male, U1 ESP32-DevKit-C, U2 LM7805_TO220, U3 MCP1754S-3302xCB, U4 MCP1825S-3.3V, U5 MCP1501-33xSN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

Commit message: Fixed PI PO, DAC port ordering, MDAT Pin, clock connection
Parts:
- added C19: 10uF, Capacitor_SMD:C_0805_2012Metric_Pad1.18x1.45mm_HandSolder, F.Cu at (137.5, 52.0)
- added C20: 0.1uF, Capacitor_SMD:C_0805_2012Metric_Pad1.18x1.45mm_HandSolder, F.Cu at (137.7, 49.0)
- added C21: 10uF, Capacitor_SMD:C_0805_2012Metric_Pad1.18x1.45mm_HandSolder, F.Cu at (134.3, 57.3)
- added C22: 0.1uF, Capacitor_SMD:C_0805_2012Metric_Pad1.18x1.45mm_HandSolder, F.Cu at (130.6, 58.8)
- added R4: 0, Resistor_SMD:R_0805_2012Metric_Pad1.20x1.40mm_HandSolder, F.Cu at (118.7, 51.3)
- added R5: 100k, Resistor_SMD:R_0805_2012Metric_Pad1.20x1.40mm_HandSolder, F.Cu at (119.9, 43.9)
- added R6: 100k, Resistor_SMD:R_0805_2012Metric_Pad1.20x1.40mm_HandSolder, F.Cu at (114.8, 57.3)
- added TP1: TestPoint, Connector_PinHeader_2.54mm:PinHeader_1x01_P2.54mm_Vertical, F.Cu at (118.2, 55.5)
Connections:
- A1 pad 19: MDAT -> MDAT1
- A1 pad 22: unconnected-(A1-Pad22) -> MDAT2
- J4 pad 1: VoutB -> VoutH
- J4 pad 11: VoutE -> VoutC
- J4 pad 13: VoutC -> VoutB
- J4 pad 3: VoutD -> VoutG
- J4 pad 7: VoutH -> VoutE
- J4 pad 9: VoutG -> VoutD
- R3 pad 1: Net-(R3-Pad1) -> ADC_CLK2
- R3 pad 2: CLK -> Net-(X1-Pad3)
- U1 pad 25: MDAT -> MDAT1
- U1 pad 28: unconnected-(U1-Pad28) -> MDAT2
- U6 pad 17: MDAT -> MDAT1
- U6 pad 18: CLK -> ADC_CLK1
- U7 pad 17: MDAT -> MDAT2
- U7 pad 18: CLK -> ADC_CLK2
- U8 pad 15: PO -> PI
- X1 pad 3: Net-(R3-Pad1) -> Net-(X1-Pad3)
Routing:
- net MDAT1: track 0.00 -> 90.8 mm, vias 0 -> 4
- net MDAT: track 75.7 -> 0.00 mm, vias 2 -> 0
- net PI: track 85.6 -> 109.0 mm
- net PO: track 114.4 -> 91.5 mm
- net CLK: track 21.6 -> 0.00 mm, vias 2 -> 0
- net ADC2_4: track 13.6 -> 28.8 mm
- net ADC2_3: track 15.3 -> 0.00 mm
- net VoutH: track 5.90 -> 11.1 mm
- net MDAT2: track 0.00 -> 5.10 mm
- net VoutE: track 9.32 -> 5.90 mm
- net VoutC: track 12.5 -> 9.32 mm
- net VoutG: track 6.40 -> 9.08 mm
- net VoutD: track 9.08 -> 6.40 mm
- net Net-(R3-Pad1): track 2.08 -> 0.00 mm
- net ADC_CLK2: track 0.00 -> 2.08 mm
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