File: hardware/board2_HV_MODULE/revised_minh_design.kicad_sch (KiCad schematic)
At the start: 18 parts, among them J1 Conn_01x07_Male, J2 Conn_01x01_Male, U1 LM7805_TO220, U2 NE5532, U3 CB101

Commit message: cleanup
Parts:
- J2: now left out of the parts list
- R1: value 10k -> 3k9
- R2: value 4.7k -> 2k
- R5, R7: value 2K -> 1k1
- R6, R8: value 1.1K -> 2k
Changed lines of the file:
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@@
     (in_bom yes) (on_board yes)
     (property "Reference" "R6" (id 0) (at 134.62 101.6 0))
-    (property "Value" "1.1K" (id 1) (at 140.97 101.6 0))
+    (property "Value" "2k" (id 1) (at 140.97 101.6 0))
     (property "Footprint" "Resistor_THT:R_Axial_DIN0207_L6.3mm_D2.5mm_P10.16mm_Horizontal" (id 2) (at 138.938 101.6 90)
       (effects (font (size 1.27 1.27)) hide)
@@
   )
   (symbol (lib_id "Connector:Conn_01x01_Male") (at 143.51 77.47 90) (unit 1)
-    (in_bom yes) (on_board yes) (fields_autoplaced)
+    (in_bom no) (on_board yes) (fields_autoplaced)
     (property "Reference" "J2" (id 0) (at 144.78 75.5649 90)
       (effects (font (size 1.27 1.27)) (justify right))
@@
     (in_bom yes) (on_board yes)
     (property "Reference" "R2" (id 0) (at 82.55 92.71 90))
-    (property "Value" "4.7k" (id 1) (at 82.55 97.79 90))
+    (property "Value" "2k" (id 1) (at 82.55 97.79 90))
     (property "Footprint" "Resistor_THT:R_Axial_DIN0207_L6.3mm_D2.5mm_P7.62mm_Horizontal" (id 2) (at 82.55 97.028 90)
       (effects (font (size 1.27 1.27)) hide)
@@
     (in_bom yes) (on_board yes)
     (property "Reference" "R8" (id 0) (at 153.67 101.6 0))
-    (property "Value" "1.1K" (id 1) (at 160.02 101.6 0))
+    (property "Value" "2k" (id 1) (at 160.02 101.6 0))
     (property "Footprint" "Resistor_THT:R_Axial_DIN0207_L6.3mm_D2.5mm_P10.16mm_Horizontal" (id 2) (at 157.988 101.6 90)
       (effects (font (size 1.27 1.27)) hide)
@@
     (in_bom yes) (on_board yes)
     (property "Reference" "R7" (id 0) (at 153.67 91.44 0))
-    (property "Value" "2K" (id 1) (at 158.75 91.44 0))
+    (property "Value" "1k1" (id 1) (at 160.02 91.44 0))
     (property "Footprint" "Resistor_THT:R_Axial_DIN0207_L6.3mm_D2.5mm_P10.16mm_Horizontal" (id 2) (at 157.988 91.44 90)
       (effects (font (size 1.27 1.27)) hide)
@@
     (in_bom yes) (on_board yes)
     (property "Reference" "R5" (id 0) (at 134.62 91.44 0))
-    (property "Value" "2K" (id 1) (at 139.7 91.44 0))
+    (property "Value" "1k1" (id 1) (at 140.97 91.44 0))
     (property "Footprint" "Resistor_THT:R_Axial_DIN0207_L6.3mm_D2.5mm_P15.24mm_Horizontal" (id 2) (at 138.938 91.44 90)
       (effects (font (size 1.27 1.27)) hide)
@@
       (effects (font (size 1.27 1.27)) (justify left))
     )
-    (property "Value" "10k" (id 1) (at 68.58 100.3299 0)
+    (property "Value" "3k9" (id 1) (at 68.58 100.3299 0)
       (effects (font (size 1.27 1.27)) (justify left))
     )
@@
     )
     (path "/b29a57d3-9503-4ca1-a1b1-94063a0f28ae"
-      (reference "R1") (unit 1) (value "10k") (footprint "Resistor_THT:R_Axial_DIN0207_L6.3mm_D2.5mm_P10.16mm_Horizontal")
+      (reference "R1") (unit 1) (value "3k9") (footprint "Resistor_THT:R_Axial_DIN0207_L6.3mm_D2.5mm_P10.16mm_Horizontal")
     )
     (path "/90448ba8-5502-4df1-8c21-bd3fac98bab5"
-      (reference "R2") (unit 1) (value "4.7k") (footprint "Resistor_THT:R_Axial_DIN0207_L6.3mm_D2.5mm_P7.62mm_Horizontal")
+      (reference "R2") (unit 1) (value "2k") (footprint "Resistor_THT:R_Axial_DIN0207_L6.3mm_D2.5mm_P7.62mm_Horizontal")
     )
     (path "/98700803-79a8-4ec2-bc5e-3326e28aa2cc"
@@
     )
     (path "/a4e2fe62-1543-4398-8850-30b5933e3401"
-      (reference "R5") (unit 1) (value "2K") (footprint "Resistor_THT:R_Axial_DIN0207_L6.3mm_D2.5mm_P15.24mm_Horizontal")
+      (reference "R5") (unit 1) (value "1k1") (footprint "Resistor_THT:R_Axial_DIN0207_L6.3mm_D2.5mm_P15.24mm_Horizontal")
     )
     (path "/494f5535-0d2a-461b-8b71-f86f3a6a73ff"
-      (reference "R6") (unit 1) (value "1.1K") (footprint "Resistor_THT:R_Axial_DIN0207_L6.3mm_D2.5mm_P10.16mm_Horizontal")
+      (reference "R6") (unit 1) (value "2k") (footprint "Resistor_THT:R_Axial_DIN0207_L6.3mm_D2.5mm_P10.16mm_Horizontal")
     )
     (path "/a2dea781-9bc1-4d50-828e-caa9d3943e1c"
-      (reference "R7") (unit 1) (value "2K") (footprint "Resistor_THT:R_Axial_DIN0207_L6.3mm_D2.5mm_P10.16mm_Horizontal")
+      (reference "R7") (unit 1) (value "1k1") (footprint "Resistor_THT:R_Axial_DIN0207_L6.3mm_D2.5mm_P10.16mm_Horizontal")
     )
     (path "/93d2ccfb-9bbb-4ea8-8868-a325feda37a0"
-      (reference "R8") (unit 1) (value "1.1K") (footprint "Resistor_THT:R_Axial_DIN0207_L6.3mm_D2.5mm_P10.16mm_Horizontal")
+      (reference "R8") (unit 1) (value "2k") (footprint "Resistor_THT:R_Axial_DIN0207_L6.3mm_D2.5mm_P10.16mm_Horizontal")
     )
     (path "/34ad081a-2df0-4615-aad1-bf529e317b2a"
