File: hardware/board2_HV_MODULE_15A12/revised_minh_design.kicad_pcb (KiCad board)
At the start: 2 copper layers, 100 x 56.6 mm, 25 parts, among them J1 Conn_01x07_Male, J2 Conn_01x01_Male, J3 Conn_01x02_Male, U1 LM7805_TO220, U2 NE5532, U4 15A12

Commit message: cleanup
Parts:
- R1: value 10k -> 4.7k
- R2: value 4.7k -> 2k
- R5, R7: value 2K -> 3.9K
- moved R3 10.3 mm to (180.8, 53.7), turned to 180 degrees
Connections:
- R3 pad 1: SGND -> VPGM
- R3 pad 2: VPGM -> SGND
Changed lines of the file:
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@@
       (effects (font (size 1 1) (thickness 0.15)))
     )
-    (fp_text value "10k" (at 5.08 2.37 90) (layer "F.Fab")
+    (fp_text value "4.7k" (at 5.08 2.37 90) (layer "F.Fab")
       (effects (font (size 1 1) (thickness 0.15)))
     )
@@
       (effects (font (size 1 1) (thickness 0.15)))
     )
-    (fp_text value "2K" (at 5.08 2.37) (layer "F.Fab")
+    (fp_text value "3.9K" (at 5.08 2.37) (layer "F.Fab")
       (effects (font (size 1 1) (thickness 0.15)))
     )
@@
       (effects (font (size 1 1) (thickness 0.15)))
     )
-    (fp_text value "2K" (at 5.08 2.37 90) (layer "F.Fab")
+    (fp_text value "3.9K" (at 5.08 2.37 90) (layer "F.Fab")
       (effects (font (size 1 1) (thickness 0.15)))
     )
@@
     )
     (fp_rect (start -3.2 34.996) (end 116.2 -3.804) (layer "F.SilkS") (width 0.12) (fill none))
+    (fp_circle (center 17.78 1.27) (end 19.576051 1.27) (layer "F.SilkS") (width 0.12) (fill none))
     (fp_circle (center 17.78 29.21) (end 19.576051 29.21) (layer "F.SilkS") (width 0.12) (fill none))
-    (fp_circle (center 17.78 1.27) (end 19.576051 1.27) (layer "F.SilkS") (width 0.12) (fill none))
-    (fp_circle (center 102.5 29.7) (end 105.41 29.7) (layer "Edge.Cuts") (width 0.12) (fill none))
+    (pad "" thru_hole circle (at 102.5 29.7 180) (size 1.524 1.524) (drill 6) (layers *.Cu *.Mask))
     (pad "1" thru_hole circle (at 0 -0.004 180) (size 1.524 1.524) (drill 0.762) (layers *.Cu *.Mask)
       (net 17 "SGND") (pinfunction "DC_INPUT_POWER_GROUND") (pintype "input"))
@@
   )
   (footprint "Resistor_THT:R_Axial_DIN0207_L6.3mm_D2.5mm_P10.16mm_Horizontal" (layer "F.Cu")
-    (at 170.561 53.721)
+    (at 180.848 53.721 180)
     (descr "Resistor, Axial_DIN0207 series, Axial, Horizontal, pin pitch=10.16mm, 0.25W = 1/4W, length*diameter=6.3*2.5mm^2, http://cdn-reichelt.de/documents/datenblatt/B400/1_4W%23YAG.pdf")
     (tags "Resistor Axial_DIN0207 series Axial Horizontal pin pitch 10.16mm 0.25W = 1/4W length 6.3mm diameter 2.5mm")
@@
     (fp_line (start 1.93 1.25) (end 8.23 1.25) (layer "F.Fab") (width 0.1))
     (fp_line (start 8.23 -1.25) (end 1.93 -1.25) (layer "F.Fab") (width 0.1))
-    (pad "1" thru_hole circle (at 0 0) (size 1.6 1.6) (drill 0.8) (layers *.Cu *.Mask)
+    (pad "1" thru_hole circle (at 0 0 180) (size 1.6 1.6) (drill 0.8) (layers *.Cu *.Mask)
+      (net 5 "VPGM") (pintype "passive"))
+    (pad "2" thru_hole oval (at 10.16 0 180) (size 1.6 1.6) (drill 0.8) (layers *.Cu *.Mask)
       (net 17 "SGND") (pintype "passive"))
-    (pad "2" thru_hole oval (at 10.16 0) (size 1.6 1.6) (drill 0.8) (layers *.Cu *.Mask)
-      (net 5 "VPGM") (pintype "passive"))
     (model "${KICAD6_3DMODEL_DIR}/Resistor_THT.3dshapes/R_Axial_DIN0207_L6.3mm_D2.5mm_P10.16mm_Horizontal.wrl"
       (offset (xyz 0 0 0))
@@
       (effects (font (size 1 1) (thickness 0.15)))
     )
-    (fp_text value "4.7k" (at 3.81 2.37 -90) (layer "F.Fab")
+    (fp_text value "2k" (at 3.81 2.37 -90) (layer "F.Fab")
       (effects (font (size 1 1) (thickness 0.15)))
     )
@@
     (property "Sheetfile" "revised_minh_design.kicad_sch")
     (property "Sheetname" "")
-    (attr exclude_from_pos_files)
+    (property "exclude_from_bom" "")
+    (attr exclude_from_pos_files exclude_from_bom)
     (fp_text reference "J2" (at 0 2.47 90) (layer "B.SilkS")
       (effects (font (size 1 1) (thickness 0.15)) (justify mirror))
@@
     (property "Sheetname" "")
     (attr through_hole)
-    (fp_text reference "J1" (at -1.27 2.77) (layer "B.SilkS")
-      (effects (font (size 1 1) (thickness 0.15)) (justify mirror))
+    (fp_text reference "J1" (at 0.2086 -12.6192) (layer "F.SilkS")
+      (effects (font (size 1 1) (thickness 0.15)))
     )
     (fp_text value "Conn_01x07_Male" (at -1.27 -12.93) (layer "B.Fab")
@@
   )
   (gr_line (start 90.424 24.638) (end 90.424 78.73) (layer "Edge.Cuts") (width 0.1))
-  (gr_arc (start 91.562 80) (mid 90.729974 79.600688) (end 90.424 78.73) (layer "Edge.Cuts") (width 0.15))
+  (gr_arc (start 91.562 80) (mid 90.729972 79.60069) (end 90.424 78.73) (layer "Edge.Cuts") (width 0.15))
   (gr_line (start 189.120974 23.368) (end 91.689 23.368) (layer "Edge.Cuts") (width 0.15))
-  (gr_arc (start 190.4 78.730968) (mid 190.031165 79.625463) (end 189.139032 80) (layer "Edge.Cuts") (width 0.15))
-  (gr_arc (start 189.120974 23.368) (mid 190.022193 23.739425) (end 190.4 24.638) (layer "Edge.Cuts") (width 0.15))
+  (gr_arc (start 190.4 78.730968) (mid 190.031168 79.625473) (end 189.139032 80) (layer "Edge.Cuts") (width 0.15))
+  (gr_arc (start 189.120974 23.368) (mid 190.022204 23.739422) (end 190.4 24.638) (layer "Edge.Cuts") (width 0.15))
   (gr_line (start 91.562 80) (end 189.139032 80) (layer "Edge.Cuts") (width 0.1))
   (gr_line (start 190.4 78.730968) (end 190.4 24.638) (layer "Edge.Cuts") (width 0.1))
-  (gr_arc (start 90.424 24.638) (mid 90.794208 23.741744) (end 91.689 23.368) (layer "Edge.Cuts") (width 0.15))
+  (gr_arc (start 90.424 24.638) (mid 90.794204 23.741737) (end 91.689 23.368) (layer "Edge.Cuts") (width 0.15))
   (gr_text "15A12" (at 125.8824 29.1084) (layer "B.SilkS")
     (effects (font (size 6 6) (thickness 1)) (justify left mirror))
@@
   (segment (start 180.771911 76.987511) (end 181.7116 77.9272) (width 1.5) (layer "F.Cu") (net 1))
   (segment (start 171.577 74.168) (end 174.935 74.168) (width 1.5) (layer "F.Cu") (net 1))
-  (segment (start 171.196 50.84) (end 171.109 50.927) (width 1.5) (layer "F.Cu") (net 2))
+  (segment (start 171.186 48.123) (end 171.069 48.24) (width 1.5) (layer "F.Cu") (net 2))
   (segment (start 175.4632 64.77) (end 175.4632 68.5598) (width 1.5) (layer "F.Cu") (net 2))
-  (segment (start 171.109 50.927) (end 171.109 51.6782) (width 1.5) (layer "F.Cu") (net 2))
   (segment (start 173.101 62.4078) (end 175.4632 64.77) (width 1.5) (layer "F.Cu") (net 2))
-  (segment (start 171.109 51.6782) (end 173.101 53.6702) (width 1.5) (layer "F.Cu") (net 2))
-  (segment (start 173.101 53.6702) (end 173.101 62.4078) (width 1.5) (layer "F.Cu") (net 2))
+  (segment (start 171.109 50.927) (end 171.196 50.927) (width 1.5) (layer "F.Cu") (net 2))
+  (segment (start 173.101 52.832) (end 173.101 62.4078) (width 1.5) (layer "F.Cu") (net 2))
+  (segment (start 171.196 50.927) (end 173.101 52.832) (width 1.5) (layer "F.Cu") (net 2))
   (segment (start 175.4632 68.5598) (end 174.935 69.088) (width 1.5) (layer "F.Cu") (net 2))
-  (segment (start 171.196 48.133) (end 171.196 50.84) (width 1.5) (layer "F.Cu") (net 2))
-  (segment (start 171.186 48.123) (end 171.196 48.133) (width 1.5) (layer "F.Cu") (net 2))
+  (segment (start 171.069 50.887) (end 171.109 50.927) (width 1.5) (layer "F.Cu") (net 2))
+  (segment (start 171.069 48.24) (end 171.069 50.887) (width 1.5) (layer "F.Cu") (net 2))
   (segment (start 185.2676 33.9394) (end 185.3134 33.9852) (width 1) (layer "F.Cu") (net 3))
   (segment (start 185.3134 33.9852) (end 188.2648 33.9852) (width 1) (layer "F.Cu") (net 3))
@@
   (segment (start 117.983 34.417) (end 120.65 31.75) (width 1.5) (layer "F.Cu") (net 8))
   (segment (start 120.65 31.75) (end 155.448 31.75) (width 1.5) (layer "F.Cu") (net 8))
-  (segment (start 171.45 26.543) (end 171.4754 26.5684) (width 1) (layer "F.Cu") (net 8))
   (segment (start 171.45 26.543) (end 171.4246 26.5684) (width 1.5) (layer "F.Cu") (net 8))
   (segment (start 117.983 41.91) (end 117.983 34.417) (width 1.5) (layer "F.Cu") (net 8))

Commit message: Used 2nd opamp for unity gain on VMON
Parts:
- R4: value 1K -> 2.2k
- R5, R7: value 3.9K -> 3k9
- R6, R8: value 1.1K -> 1k1
Connections:
- R5 pad 1: VMON_3V3 -> VMON_OPAMP
- R6 pad 2: VMON_3V3 -> VMON_OPAMP
- U2 pad 5: unconnected-(U2-Pad5) -> VMON_OPAMP
- U2 pad 6: unconnected-(U2-Pad6) -> VMON_3V3
- U2 pad 7: unconnected-(U2-Pad7) -> VMON_3V3
Routing:
- net VMON_OPAMP: track 0.00 -> 7.21 mm
- net VMON_3V3: track 36.8 -> 31.0 mm

Commit message: added BOM Excel
Changed lines of the file:
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@@
   (segment (start 171.186 36.967) (end 171.45 36.703) (width 0.5) (layer "B.Cu") (net 10))
   (segment (start 171.186 40.503) (end 171.186 36.967) (width 0.5) (layer "B.Cu") (net 10))
-  (segment (start 185.3892 61.946) (end 185.5416 61.946) (width 0.8) (layer "F.Cu") (net 11))
   (segment (start 171.186 43.043) (end 171.186 45.583) (width 0.5) (layer "F.Cu") (net 11))
   (segment (start 175.3062 61.8952) (end 185.5924 61.8952) (width 0.5) (layer "B.Cu") (net 11))
